File: pcb/battle-bot.kicad_sch (KiCad schematic)
At the start: 18 parts, among them J1 Conn_01x02_Pin, J2 Conn_01x02_Pin, Q1 PMOS, Q2 PMOS, U1 TPS5430DDA, U2 STM32H503RBTx

Commit message: Save
Parts:
- removed U2: STM32H503RBTx, Package_QFP:LQFP-64_10x10mm_P0.5mm, symbol MCU_ST_STM32H5:STM32H503RBTx
- added U2: STM32G474VETx, Package_QFP:LQFP-100_14x14mm_P0.5mm, symbol MCU_ST_STM32G4:STM32G474VETx
Connections:
- net +3V3 is gone; now on net +5V: C5.1, C6.1, L1.2, R1.1
- new net: U2.23 (VSS), U2.48 (VSS), U2.63 (VSS), U2.74 (VSS), U2.99 (VSS)
Other:
- note added: "C2653814"
- note added: "C3289450"

Commit message: Finish drivers
Parts:
- removed D1, D2: D, symbol Device:D
- removed D3: B5819W, Diode_SMD:D_SOD-123, symbol Device:D_Schottky
- removed Q1, Q2: PMOS, symbol Simulation_SPICE:PMOS
- removed U1: TPS5430DDA, Package_SO:TI_SO-PowerPAD-8_ThermalVias, symbol Regulator_Switching:TPS5430DDA
- removed U2: STM32G474VETx, Package_QFP:LQFP-100_14x14mm_P0.5mm, symbol MCU_ST_STM32G4:STM32G474VETx
- added AE1: Antenna, RF_Antenna:Johanson_2450AT18x100, symbol Device:Antenna
- added C10: 100n, Resistor_SMD:R_0402_1005Metric, symbol Device:C
- added C11, C14, C16, C17: 47u, Capacitor_SMD:C_1206_3216Metric, symbol Device:C
- added C12, C27: 10n, Capacitor_SMD:C_0402_1005Metric, symbol Device:C
- added C13: 33n, Capacitor_SMD:C_0402_1005Metric, symbol Device:C
- added C15: 1n, Capacitor_SMD:C_0402_1005Metric, symbol Device:C
- added C18: 220u, Capacitor_THT:C_Radial_D6.3mm_H7.0mm_P2.50mm, symbol Device:C
- added C19: 2n2, Capacitor_SMD:C_0603_1608Metric, symbol Device:C
- added C20, C23: 12p, Capacitor_SMD:C_0402_1005Metric, symbol Device:C
- added C21: 4p7, Capacitor_SMD:C_0603_1608Metric, symbol Device:C
- added C22: 1p5, Capacitor_SMD:C_0402_1005Metric, symbol Device:C
- added C24: 1p, Capacitor_SMD:C_0402_1005Metric, symbol Device:C
- added C25, C8: 10u, Resistor_SMD:R_0402_1005Metric, symbol Device:C
- added C26: 4u7, Capacitor_SMD:C_0402_1005Metric, symbol Device:C
- added C28: 220p, Resistor_SMD:R_0402_1005Metric, symbol Device:C
- added C29, C30, C9: 100n, Capacitor_SMD:C_0402_1005Metric, symbol Device:C
- added C31: 0p3, Capacitor_SMD:C_0402_1005Metric, symbol Device:C
- added C62: C, Capacitor_SMD:C_0402_1005Metric, symbol Device:C
- added C63, C64, C65, C66: 2m2, symbol Device:C
- added C7: 100u, Resistor_SMD:R_1206_3216Metric, symbol Device:C
- added D1: LEDG, LED_SMD:LED_0603_1608Metric, symbol Device:LED
- added L2: 2n7, Inductor_SMD:L_0402_1005Metric, symbol Device:L
- added L3: 8n2, Inductor_SMD:L_0402_1005Metric, symbol Device:L
- added L4: 3n9, Inductor_SMD:L_0402_1005Metric, symbol Device:L
- added Q1: AO3400A, Package_TO_SOT_SMD:SOT-23, symbol Transistor_FET:AO3400A
- added R10, R11, R9: 1k, Resistor_SMD:R_0402_1005Metric, symbol Device:R
- added R12, R6: 22k, Resistor_SMD:R_0402_1005Metric, symbol Device:R
- added R3, R4, R8: 100k, Resistor_SMD:R_0402_1005Metric, symbol Device:R
- added R39, R40: R, Resistor_SMD:R_0402_1005Metric, symbol Device:R
- added R5: 15k, Resistor_SMD:R_0402_1005Metric, symbol Device:R
- added R7: 10k, Resistor_SMD:R_0402_1005Metric, symbol Device:R
- added U1: TPS53319, Package_DFN_QFN:DFN-22-1EP_5x6mm_P0.5mm_EP3.14x4.3mm, symbol User_Symbols:TPS53319
- added U14: AMS1117-3.3, Package_TO_SOT_SMD:SOT-223-3_TabPin2, symbol Regulator_Linear:AMS1117-3.3
- added U2: nRF24L01P, Package_DFN_QFN:QFN-20-1EP_4x4mm_P0.5mm_EP2.5x2.5mm, symbol RF:nRF24L01P
- added U3: AT2401C, Package_DFN_QFN:QFN-16-1EP_3x3mm_P0.5mm_EP1.7x1.7mm, symbol User_Symbols:AT2401C
- added U4: ICM-42688-P, Package_LGA:LGA-14_3x2.5mm_P0.5mm_LayoutBorder3x4y, symbol Symbols:ICM-42688-P
- added U5: LFL152G45TC1A219, User_Footprints:LFL152G45TC1A219, symbol User_Symbols:LFL152G45TC1A219
- added U6: STM32G431RBTx, Package_QFP:LQFP-64_10x10mm_P0.5mm, symbol MCU_ST_STM32G4:STM32G431RBTx
- added Y1: 16MHz, Crystal:Crystal_SMD_3225-4Pin_3.2x2.5mm, symbol Device:Crystal_GND24
- C1, C2: footprint Capacitor_SMD:C_1206_3216Metric -> Capacitor_SMD:C_0805_2012Metric; LCSC C12891 -> C45783
- C3: value 10n -> 22u; footprint Capacitor_SMD:C_0402_1005Metric -> Capacitor_SMD:C_0805_2012Metric; LCSC C15195 -> C45783
- C4: value 47u -> 22u; footprint Capacitor_SMD:C_1206_3216Metric -> Capacitor_SMD:C_0805_2012Metric; LCSC C96123 -> C45783
- C5, C6: value 47u -> 1u; footprint Capacitor_SMD:C_1206_3216Metric -> Capacitor_SMD:C_0402_1005Metric; LCSC C96123 -> C52923
- J1, J2: LCSC (none) -> C431092
- L1: value 15u -> 1u; footprint Inductor_SMD:L_Changjiang_FNR6020S -> Inductor_SMD:L_Changjiang_FXL0630; LCSC C168015 -> C167216
- R1: value R -> 22k; LCSC C25744 -> C25768
- R2: value R -> 10k; LCSC C25890 -> C25744
Connections:
- net BT is gone; now on net VDD: C3.1
- net +5V: now also C11.1, C14.1, C16.1, C17.1, C18.1, D1.2 (A), R39.1, R40.1, R8.1; no longer C4.1, C5.1, C6.1, R1.1
- net GND: now also C3.2, R2.1, C10.2, C11.2, C12.2, C13.2, C14.2, C15.2, C16.2, C17.2, C18.2, C19.1, C20.1, C21.2, C23.2, C24.2, C25.2, C26.2, C27.2, C28.2, C29.2, C30.2, C31.2, C62.2, C63.2, C64.2, C65.2, C66.2, C7.2, C8.2, Q1.2 (S), R12.2, R3.2, R4.2, R5.2, R6.2, U1.23 (GND), U1.5 (ROVP), U2.14 (VSS), U2.17 (VSS), U2.20 (VSS), U2.21 (PAD), U2.8 (VSS), U3.1 (GND), U3.11 (GND), U3.12 (GND), U3.15 (GND), U3.17 (GND), U3.2 (GND), U3.3 (GND), U3.7 (GND), U3.8 (GND), U3.9 (GND), U4.11 (RESV), U4.6 (GND), U4.7 (RESV), U5.1 (GND), U5.3 (GND), U6.15 (VSS), U6.27 (VSSA), U6.31 (VSS), U6.47 (VSS), U6.63 (VSS), Y1.2, Y1.4; no longer R2.2
- net VDD: now also C1.1, C2.1, C4.1, C5.1, J1.1 (Pin_1), J2.1 (Pin_1), R1.2, C63.1, C64.1, C65.1, C66.1, U1.12 (VIN), U1.13 (VIN), U1.14 (VIN), U1.15 (VIN), U1.16 (VIN), U1.17 (VIN), U1.19 (VDD)
- net at L1.1: now also C9.1, U1.10 (LL), U1.11 (LL), U1.6 (LL), U1.7 (LL), U1.8 (LL), U1.9 (LL); no longer C3.2
- removed net VSNS: R1.2, R2.1
- new net: R3.1, U1.21 (TRIP)
- new net: R11.2, U3.5 (TXEN)
- new net: R10.1, R12.1, U3.6 (RXEN)
- new net: C31.1, U3.10 (ANT), U5.4 (IN)
- new net: R7.2, R8.2
- new net: R5.1, R7.1, U1.1 (VFB)
- new net: C6.1, U1.18 (VREG)
- new net: R4.1, U1.20 (MODE)
- new net: C9.2, U1.4 (VBST)
- new net: R6.1, U2.16 (IREF)
- new net: C62.1, Q1.1 (G), R40.2
- new net: L3.1, L4.1, U2.13 (ANT2)
- new net: L2.1, L3.2, U2.12 (ANT1)
- new net: C22.2, C24.1, U3.4 (TXRX)
- new net: AE1.1 (A), U5.2 (OUT)
- new net: C22.1, L4.2
- new net: C13.1, U2.19 (DVDD)
- new net: D1.1 (K), R9.1
- new net +3V3: C10.1, C12.1, C15.1, C25.1, C26.1, C27.1, C28.1, C29.1, C30.1, C7.1, C8.1, U2.15 (VDD), U2.18 (VDD), U2.7 (VDD), U3.14 (VDD), U3.16 (VDD), U4.5 (VDDIO), U4.8 (VDD)
- new net CAL: Q1.3 (D), R39.2
- new net CE: R10.2
- new net CLK: U2.3 (SCK), U4.13 (CLK)
- new net GCS: U4.12 (CS)
- new net GINT: U4.4 (INT1)
- new net MISO: U2.5 (MISO), U4.1 (SDO)
- new net MOSI: U2.4 (MOSI), U4.14 (SDI)
- new net PGD: R9.2, U1.3 (PGD)
- new net RCE: U2.1 (CE)
- new net RCS: U2.2 (CSN)
- new net REN: R1.1, R2.2, U1.2 (EN)
- new net RIRQ: U2.6 (IRQ)
- new net VPA: C19.2, C21.1, L2.2, R11.1, U2.11 (VDD_PA)
- new net XC1: C23.1, U2.10 (XC1), Y1.1
- new net XC2: C20.2, U2.9 (XC2), Y1.3
- no-connect marks 1 -> 2
Other:
- added sheet LargeMotor (large-motor.kicad_sch)
- added sheet SmallMotor1 (small-motor.kicad_sch)
- added sheet SmallMotor2 (small-motor.kicad_sch)
- added sheet SmallMotor3 (small-motor.kicad_sch)
- note added: "Batteries"
- note added: "Bulk Capacitance"
- note added: "C25838715"
- note added: "Caps and Connectors"
- note added: "IMU"
- note added: "KTH5702AQ3QNS"
- note added: "LP38690SD-3.3/NOPB"
- note added: "NRF24"
- note added: "Regulator"
- note added: "SENSORS"
- note removed: "C2653814"
- note removed: "C3289450"
- moved on the sheet: J1, J2

Commit message: Finish rough layout
Parts:
- removed J2: Conn_01x02_Pin, Connector_AMASS:AMASS_XT30PW-M_1x02_P2.50mm_Horizontal, symbol Connector:Conn_01x02_Pin
- removed Q1: AO3400A, Package_TO_SOT_SMD:SOT-23, symbol Transistor_FET:AO3400A
- removed U14: AMS1117-3.3, Package_TO_SOT_SMD:SOT-223-3_TabPin2, symbol Regulator_Linear:AMS1117-3.3
- added C67: C, Capacitor_SMD:C_0402_1005Metric, symbol Device:C
- added C68: 2m2, Capacitor_THT:C_Radial_D10.0mm_H16.0mm_P5.00mm, symbol Device:C
- added C73: 2u2, Capacitor_SMD:C_0402_1005Metric, symbol Device:C
- added C74, C75: 100n, Capacitor_SMD:C_0402_1005Metric, symbol Device:C
- added C76: 10u, Capacitor_SMD:C_0603_1608Metric, symbol Device:C
- added C93: 10u, Resistor_SMD:R_0402_1005Metric, symbol Device:C
- added J2: Conn_01x04_MountingPin, Connector_JST:JST_GH_SM04B-GHS-TB_1x04-1MP_P1.25mm_Horizontal, symbol Connector_Generic_MountingPin:Conn_01x04_MountingPin
- added Q2: AO3401A, Package_TO_SOT_SMD:SOT-23, symbol Transistor_FET:AO3401A
- added R41: 1k, Resistor_SMD:R_0402_1005Metric, symbol Device:R
- added R42: R, Resistor_SMD:R_0402_1005Metric, symbol Device:R
- added U15: LP38690SD, Package_DFN_QFN:DFN-6-1EP_3x3mm_P0.95mm_EP1.7x2.6mm, symbol User_Symbols:LP38690SD-3.3
- C62: value C -> 2m2; footprint Capacitor_SMD:C_0402_1005Metric -> Capacitor_THT:C_Radial_D10.0mm_H16.0mm_P5.00mm; LCSC (none) -> C5438720
- C63, C64, C65, C66: footprint (none) -> Capacitor_THT:C_Radial_D10.0mm_H16.0mm_P5.00mm; LCSC (none) -> C5438720
- R39, R40: value R -> 2k2; LCSC (none) -> C25879
Connections:
- net +3V3: now also R39.1, R40.1, C93.1, J2.1 (Pin_1)
- net +5V: now also C74.1, C76.1, Q2.2 (S), R42.1, U15.1 (IN), U15.6 (IN); no longer R39.1, R40.1
- net CAL: now also Q2.3 (D), R41.1; no longer R39.2
- net ESCL: now also R40.2, J2.3 (Pin_3)
- net ESDA: now also R39.2, J2.2 (Pin_2)
- net GND: now also C67.2, C68.2, C73.2, C74.2, C75.2, C76.2, C93.2, J2.4 (Pin_4), J2.MP (MountPin), R41.2, U15.2 (GND), U15.7 (PAD)
- net VDD: now also C62.1, C68.1
- new net: C67.1, Q2.1 (G), R42.2
- new net VDDRF: C73.1, C75.1, U15.4 (OUT), U15.5 (SNS)
Other:
- note added: "Battery"
- note added: "Buck Regulator"
- note added: "Bulk Capacitors"
- note added: "Calibrate"
- note added: "Connectors"
- note added: "Low Noise LDO"
- note added: "Sensors"
- note removed: "Batteries"
- note removed: "Bulk Capacitance"
- note removed: "Caps and Connectors"
- note removed: "LP38690SD-3.3/NOPB"
- note removed: "Regulator"
- note removed: "SENSORS"
- moved on the sheet: C26, C29, C30, J1, U4, U6

Commit message: Save layout
Parts:
- removed AE1: Antenna, RF_Antenna:Johanson_2450AT18x100, symbol Device:Antenna
- removed C64: 2m2, Capacitor_THT:C_Radial_D10.0mm_H16.0mm_P5.00mm, symbol Device:C
- removed J1: Conn_01x02_Pin, Connector_AMASS:AMASS_XT30PW-M_1x02_P2.50mm_Horizontal, symbol Connector:Conn_01x02_Pin
- added AE1: Antenna_Chip, RF_Antenna:Johanson_2450AT18x100, symbol Device:Antenna_Chip
- added J1, J12: Conn_01x01_Pin, MountingHole:MountingHole_3.2mm_M3_Pad_Via, symbol Connector:Conn_01x01_Pin
- C62, C65, C66, C68: footprint Capacitor_THT:C_Radial_D10.0mm_H16.0mm_P5.00mm -> User_Footprints:C_D10xL16_Horizontal
- C63: value 2m2 -> 100n; footprint Capacitor_THT:C_Radial_D10.0mm_H16.0mm_P5.00mm -> Capacitor_SMD:C_0402_1005Metric; LCSC C5438720 -> C1525
Connections:
- net +5V: now also C63.1
- net GND: now also C65.1, C68.1, J1.1 (Pin_1); no longer C65.2, C68.2
- net VDD: now also C65.2, C68.2, J12.1 (Pin_1); no longer C63.1, C65.1, C68.1
- net at U5.2 (OUT): now also AE1.1 (FEED)
- no-connect marks 2 -> 3
Other:
- note added: "UVLO"
- moved on the sheet: C68, C73, C74, C75, C76, U15

Commit message: Save old buck regulator
Parts:
- removed J2: Conn_01x04_MountingPin, Connector_JST:JST_GH_SM04B-GHS-TB_1x04-1MP_P1.25mm_Horizontal, symbol Connector_Generic_MountingPin:Conn_01x04_MountingPin
- removed U4: ICM-42688-P, Package_LGA:LGA-14_3x2.5mm_P0.5mm_LayoutBorder3x4y, symbol Symbols:ICM-42688-P
- added C64, C69: 12p, Capacitor_SMD:C_0402_1005Metric, symbol Device:C
- added C72, C78: 2m2, User_Footprints:C_D10xL16_Horizontal, symbol Device:C
- added C79, C80: 10n, Capacitor_SMD:C_0402_1005Metric, symbol Device:C
- added C81, C82, C83, C84, C87, C92: 100n, Capacitor_SMD:C_0402_1005Metric, symbol Device:C
- added C85, C86, C94: 1u, Capacitor_SMD:C_0402_1005Metric, symbol Device:C
- added C88, C89, C90, C91: 47u, Capacitor_SMD:C_1206_3216Metric, symbol Device:C
- added C95, C96: 22u, Capacitor_SMD:C_0805_2012Metric, symbol Device:C
- added D5: LEDG, LED_SMD:LED_0603_1608Metric, symbol Device:LED
- added FB1: FerriteBead, Inductor_SMD:L_0805_2012Metric, symbol Device:FerriteBead
- added J13: Conn_ARM_SWD_TagConnect_TC2030-NL, Connector:Tag-Connect_TC2030-IDC-NL_2x03_P1.27mm_Vertical, symbol Connector:Conn_ARM_SWD_TagConnect_TC2030-NL
- added L5: 2u2, Inductor_SMD:L_Chilisin_BMRB00060618, symbol Device:L
- added R43, R47: 1k, Resistor_SMD:R_0402_1005Metric, symbol Device:R
- added R44: 15k, Resistor_SMD:R_0402_1005Metric, symbol Device:R
- added R45: 2k2, Resistor_SMD:R_0402_1005Metric, symbol Device:R
- added R46: 1k2, Resistor_SMD:R_0402_1005Metric, symbol Device:R
- added R48: 330k, symbol Device:R
- added R61: 15k, symbol Device:R
- added U1: TPS56C230, Package_DFN_QFN:VQFN-20-1EP_3x3mm_P0.45mm_EP1.55x1.55mm, symbol User_Symbols:TPS56C230
- added U4: ICM-42688-P, Package_LGA:LGA-14_3x2.5mm_P0.5mm_LayoutBorder3x4y, symbol User_Symbols:ICM-42688-P
- added Y2: 16MHz, Crystal:Crystal_SMD_3225-4Pin_3.2x2.5mm, symbol Device:Crystal_GND24
- C10: value 100n -> 10u; footprint Resistor_SMD:R_0402_1005Metric -> Capacitor_SMD:C_0402_1005Metric; LCSC C1525 -> C15525
- C25, C28: footprint Resistor_SMD:R_0402_1005Metric -> Capacitor_SMD:C_0402_1005Metric
- C67: value C -> 4u7; LCSC (none) -> C23733
- C7: footprint Resistor_SMD:R_1206_3216Metric -> Capacitor_SMD:C_1206_3216Metric
- C73: value 2u2 -> 10u; LCSC C12530 -> C15525
- C8: value 10u -> 1u; footprint Resistor_SMD:R_0402_1005Metric -> Capacitor_SMD:C_0402_1005Metric; LCSC C15525 -> C52923
- C93: value 10u -> 100n; footprint Resistor_SMD:R_0402_1005Metric -> Capacitor_SMD:C_0402_1005Metric; LCSC C15525 -> C307331
- L1: value 1u -> 2u2
- R1: value 22k -> 100k; LCSC C25768 -> C25741
- R39: value 2k2 -> 10k; LCSC C25879 -> C25744
- R40: value 2k2 -> 8k6; LCSC C25879 -> C25744
- R42: value R -> 100k; LCSC (none) -> C25741
- R5: value 15k -> 1k2
- R7: value 10k -> 8k6
- R8: value 100k -> 1k5; footprint Resistor_SMD:R_0402_1005Metric -> (none); LCSC C25741 -> (none)
- renumbered U5 to FL1
Connections:
- net CE is gone; now on net RCE: R10.2
- net VDDRF is gone; now on net +3V3: C73.1, C75.1, U15.4 (OUT), U15.5 (SNS)
- net +3V3: now also U6.16 (VDD), U6.32 (VDD), U6.48 (VDD), U6.64 (VDD), C79.1, C80.1, C81.1, C82.1, C83.1, C86.1, C87.1, FB1.2, J13.1 (VCC), U4.5 (VDDIO), U4.8 (VDD); no longer C93.1, R39.1, R40.1
- net +5V: now also R40.1, R7.1, C88.1, C89.1, C90.1, C91.1, D5.2 (A), L5.2; no longer R8.1
- net CLK: now also U6.35 (PB13), U4.13 (CLK)
- net CPA1: now also U6.34 (PB12)
- net CPA2: now also U6.21 (PA7)
- net CPA3: now also U6.26 (PB2)
- net CPB1: now also U6.36 (PB14)
- net CPB2: now also U6.22 (PC4)
- net CPB3: now also U6.11 (PC3)
- net CPC1: now also U6.37 (PB15)
- net CPC2: now also U6.23 (PC5)
- net CPC3: now also U6.33 (PB11)
- net GCS: now also U6.43 (PA9), U4.12 (CS)
- net GINT: now also U6.3 (PC14), U4.4 (INT1)
- net GND: now also R8.2, C64.1, C69.1, C72.1, C78.2, C79.2, C80.2, C81.2, C82.2, C83.2, C84.2, C85.2, C86.2, C87.2, C88.2, C89.2, C90.2, C91.2, C94.2, C95.2, C96.2, J13.5 (GND), R45.2, R46.2, R61.2, U1.10 (NC), U1.13 (AGND), U1.16 (NC), U1.18 (PGND), U1.21 (PAD), U1.7 (PGND), U1.8 (PGND), U4.11 (RESV), U4.6 (GND), U4.7 (RESV), Y2.2, Y2.4; no longer U1.5 (ROVP)
- net INHA1: now also U6.58 (PB5)
- net INHA2: now also U6.38 (PC6)
- net INHA3: now also U6.59 (PB6)
- net INHB1: now also U6.56 (PB3)
- net INHB2: now also U6.39 (PC7)
- net INHB3: now also U6.60 (PB7)
- net INHC1: now also U6.30 (PB10)
- net INHC2: now also U6.40 (PC8)
- net INHC3: now also U6.61 (PB8)
- net INLA1: now also U6.41 (PC9)
- net INLA2: now also U6.57 (PB4)
- net INLA3: now also U6.55 (PD2)
- net INLB1: now also U6.62 (PB9)
- net INLB2: now also U6.52 (PC10)
- net INLB3: now also U6.4 (PC15)
- net INLC1: now also U6.53 (PC11)
- net INLC2: now also U6.54 (PC12)
- net INLC3: now also U6.51 (PA15)
- net MISO: now also U6.44 (PA10), U4.1 (SDO)
- net MOSI: now also U6.45 (PA11), U4.14 (SDI)
- net PGD: now also R47.2, U1.9 (PGD)
- net RCE: now also U6.46 (PA12)
- net RCS: now also U6.42 (PA8)
- net REN: now also R1.2; no longer R1.1
- net RIRQ: now also U6.7 (PG10)
- net SO1: now also U6.12 (PA0)
- net SO2: now also U6.13 (PA1)
- net SO3: now also U6.14 (PA2)
- net VDD: now also C93.1, R1.1, C72.2, C78.1, C95.1, C96.1, R44.1, U1.2 (VIN), U1.3 (VIN), U1.4 (VIN), U1.5 (VIN); no longer R1.2
- net WCPA: now also U6.18 (PA4)
- net WCPB: now also U6.19 (PA5)
- net WCPC: now also U6.20 (PA6)
- net WHA: now also U6.8 (PC0)
- net WHB: now also U6.9 (PC1)
- net WHC: now also U6.10 (PC2)
- net WLA: now also U6.2 (PC13)
- net WLB: now also U6.24 (PB0)
- net WLC: now also U6.25 (PB1)
- net WSO: now also U6.17 (PA3)
- net at R7.2: now also R5.1, U1.1 (VFB); no longer R8.2
- net VREG: now reaches C6.1, U1.18 (VREG)
- net VREG: now also U1.22 (RF)
- net VBAT: now reaches U6.1 (VBAT)
- net VBAT: now also R44.2, R45.1
- net +3V3A: now reaches U6.28 (VREF+)
- net +3V3A: now also U6.29 (VDDA), C84.1, C85.1, FB1.1
- net SWDIO: now reaches U6.49 (PA13)
- net SWDIO: now also J13.2 (SWDIO)
- net XTO: now reaches U6.5 (PF0)
- net XTO: now also C64.2, Y2.3
- net SWCLK: now reaches U6.50 (PA14)
- net SWCLK: now also J13.4 (SWCLK)
- net XTI: now reaches U6.6 (PF1)
- net XTI: now also R43.1
- net ESCL: no longer names the net of R40.2
- net ESCL: now also R46.1, U1.14 (FB)
- net ESDA: no longer names the net of R39.2
- net ESDA: now also U1.5 (ROVP)
- new net: C92.2, U1.1 (BST)
- new net: R48.2, U1.15 (MODE)
- new net: C94.1, R48.1, R61.1, U1.17 (VCC)
- new net: C92.1, L5.1, U1.19 (SW), U1.20 (SW), U1.6 (SW)
- new net: R39.1, R8.1
- new net: D5.1 (K), R47.1
- new net EN: U1.12 (EN)
- new net XTR: C69.2, R43.2, Y2.1
- no-connect marks 3 -> 5
Other:
- note added: "4V9 Out & 5V5 OVP"
- note removed: "C25838715"
- note removed: "Connectors"
- note removed: "KTH5702AQ3QNS"
- note removed: "Sensors"
- note removed: "UVLO"
- moved on the sheet: C1, C11, C14, C16, C17, C18, C2, C3, C4, C5, C6, C63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

Commit message: Finish pcb
Parts:
- removed C1, C2, C3, C4: 22u, Capacitor_SMD:C_0805_2012Metric, symbol Device:C
- removed C11, C14, C16, C17: 47u, Capacitor_SMD:C_1206_3216Metric, symbol Device:C
- removed C18: 220u, Capacitor_THT:C_Radial_D6.3mm_H7.0mm_P2.50mm, symbol Device:C
- removed C5, C6: 1u, Capacitor_SMD:C_0402_1005Metric, symbol Device:C
- removed C64, C69: 12p, Capacitor_SMD:C_0402_1005Metric, symbol Device:C
- removed C9: 100n, Capacitor_SMD:C_0402_1005Metric, symbol Device:C
- removed D1: LEDG, LED_SMD:LED_0603_1608Metric, symbol Device:LED
- removed R39: 10k, Resistor_SMD:R_0402_1005Metric, symbol Device:R
- removed R4: 100k, Resistor_SMD:R_0402_1005Metric, symbol Device:R
- removed R43, R9: 1k, Resistor_SMD:R_0402_1005Metric, symbol Device:R
- removed R5: 1k2, Resistor_SMD:R_0402_1005Metric, symbol Device:R
- removed R61: 15k, symbol Device:R
- removed R7: 8k6, Resistor_SMD:R_0402_1005Metric, symbol Device:R
- removed R8: 1k5, symbol Device:R
- removed U1: TPS53319, Package_DFN_QFN:DFN-22-1EP_5x6mm_P0.5mm_EP3.14x4.3mm, symbol User_Symbols:TPS53319
- removed Y2: 16MHz, Crystal:Crystal_SMD_3225-4Pin_3.2x2.5mm, symbol Device:Crystal_GND24
- AE1: LCSC C89334 -> C127629
- C13: value 33n -> 100n; LCSC C1585 -> C1525
- C19: footprint Capacitor_SMD:C_0603_1608Metric -> Capacitor_SMD:C_0402_1005Metric; LCSC C1604 -> C1531
- C21: footprint Capacitor_SMD:C_0603_1608Metric -> Capacitor_SMD:C_0402_1005Metric; LCSC C1669 -> C1569
- D5: value LEDG -> LEDW; LCSC (none) -> C2290
- L1: value 2u2 -> 6n8; footprint Inductor_SMD:L_Changjiang_FXL0630 -> Inductor_SMD:L_0402_1005Metric; LCSC C167216 -> C82919
- L4: LCSC C76775 -> C14033
- R1, R3: value 100k -> 4k7; LCSC C25741 -> C25900
- R2: value 10k -> 51k; LCSC C25744 -> C25794
- R40: value 8k6 -> 33k; LCSC C25744 -> C25779
- R46: value 1k2 -> 4k7; LCSC C25756 -> C25900
- R47: LCSC (none) -> C11702
- R48: value 330k -> 100k; footprint (none) -> Resistor_SMD:R_0402_1005Metric; LCSC (none) -> C25741
- U1: footprint Package_DFN_QFN:VQFN-20-1EP_3x3mm_P0.45mm_EP1.55x1.55mm -> User_Footprints:VQFN-20_3x3mm_P0.45
Connections:
- net XTI is gone; now on net CPA3: U6.6 (PF1)
- net XTO is gone; now on net CPC3: U6.5 (PF0)
- net +5V: no longer L1.2
- net CLK: now also U6.52 (PC10); no longer U6.35 (PB13)
- net CPA1: now also U6.14 (PA2); no longer U6.34 (PB12)
- net CPA2: now also U6.26 (PB2); no longer U6.21 (PA7)
- net CPA3: no longer U6.26 (PB2)
- net CPB1: now also U6.11 (PC3); no longer U6.36 (PB14)
- net CPB3: now also U6.9 (PC1); no longer U6.11 (PC3)
- net CPC1: now also U6.10 (PC2); no longer U6.37 (PB15)
- net CPC2: now also U6.12 (PA0); no longer U6.23 (PC5)
- net CPC3: no longer U6.33 (PB11)
- net EN: now also R2.2, R3.1
- net GCS: now also U6.55 (PD2); no longer U6.43 (PA9)
- net GINT: now also U6.57 (PB4); no longer U6.3 (PC14)
- net GND: now also C65.2, C66.1, C68.2, C72.2, R1.2; no longer C65.1, C66.2, C68.1, C72.1, R2.1
- net INHA1: now also U6.38 (PC6); no longer U6.58 (PB5)
- net INHA2: now also U6.30 (PB10); no longer U6.38 (PC6)
- net INHA3: now also U6.41 (PC9); no longer U6.59 (PB6)
- net INHB1: now also U6.39 (PC7); no longer U6.56 (PB3)
- net INHB2: now also U6.19 (PA5); no longer U6.39 (PC7)
- net INHB3: now also U6.61 (PB8); no longer U6.60 (PB7)
- net INHC1: now also U6.40 (PC8); no longer U6.30 (PB10)
- net INHC2: now also U6.17 (PA3); no longer U6.40 (PC8)
- net INHC3: now also U6.59 (PB6); no longer U6.61 (PB8)
- net INLA1: now also U6.7 (PG10); no longer U6.41 (PC9)
- net INLA2: now also U6.20 (PA6); no longer U6.57 (PB4)
- net INLA3: now also U6.62 (PB9); no longer U6.55 (PD2)
- net INLB1: now also U6.4 (PC15); no longer U6.62 (PB9)
- net INLB2: now also U6.18 (PA4); no longer U6.52 (PC10)
- net INLB3: now also U6.60 (PB7); no longer U6.4 (PC15)
- net INLC1: now also U6.3 (PC14); no longer U6.53 (PC11)
- net INLC2: now also U6.2 (PC13); no longer U6.54 (PC12)
- net INLC3: now also U6.58 (PB5); no longer U6.51 (PA15)
- net MISO: now also U6.53 (PC11); no longer U6.44 (PA10)
- net MOSI: now also U6.54 (PC12); no longer U6.45 (PA11)
- net RCS: now also U6.51 (PA15); no longer U6.42 (PA8)
- net RIRQ: now also U6.56 (PB3); no longer U6.7 (PG10)
- net SO1: now also U6.13 (PA1); no longer U6.12 (PA0)
- net SO2: now also U6.21 (PA7); no longer U6.13 (PA1)
- net SO3: now also U6.8 (PC0); no longer U6.14 (PA2)
- net VDD: now also C65.1, C66.2, C68.1, C72.1, R2.1; no longer C65.2, C66.1, C68.2, C72.2, R1.1
- net WCPA: now also U6.36 (PB14); no longer U6.18 (PA4)
- net WCPB: now also U6.33 (PB11); no longer U6.19 (PA5)
- net WCPC: now also U6.34 (PB12); no longer U6.20 (PA6)
- net WHA: now also U6.43 (PA9); no longer U6.8 (PC0)
- net WHB: now also U6.44 (PA10); no longer U6.9 (PC1)
- net WHC: now also U6.45 (PA11); no longer U6.10 (PC2)
- net WLA: now also U6.24 (PB0); no longer U6.2 (PC13)
- net WLB: now also U6.25 (PB1); no longer U6.24 (PB0)
- net WLC: now also U6.23 (PC5); no longer U6.25 (PB1)
- net WSO: now also U6.37 (PB15); no longer U6.17 (PA3)
- net at R48.2, U1.15 (MODE): now also R1.1
- net at L1.1: now also FL1.2 (OUT)
- net at AE1.1 (FEED): now also L1.2; no longer FL1.2 (OUT)
- removed net REN: R1.2, R2.2
- no-connect marks 5 -> 7
Other:
- note added: "4S LiPo UVP"
- note added: "4V8 Output"
- note added: "5V Buck"
- note removed: "4V9 Out & 5V5 OVP"
- note removed: "Buck Regulator"
- moved on the sheet: AE1, C26, C29, C30, C67, C88, C89, C90, C91, C92, C93, C94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
